File: pcb/tt06-vga-interposer/tt06-vga-interposer.kicad_pcb (KiCad board)
At the start: 2 copper layers, 72.4 x 61.6 mm, 65 parts, among them CON1 Bottom pins, CON2 Bottom pins, CON3 Top socket, CON4 Top socket, J1 Conn_02x09_Odd_Even, J2 DE15_Receptacle_HighDensity_M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, J3 Conn_01x04_Pin, J4 Conn_01x04_Pin, J5 Conn_02x07_Odd_Even, U1 OPA3355EA, U2 SN74LVC245APW

Commit message: Tidy up interposer schematic a little
Other:
- board text removed: "Mousebites for VGA breakout?"
- board text removed: "Thicker power/ground traces?"
Changed lines of the file:
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@@
-		)
-	)
-	(gr_text "Thicker power/ground traces?"
-		(at 131.445 77.089 0)
-		(layer "User.1")
-		(effects
-			(font
-				(size 1 1)
-				(thickness 0.1)
-			)
-			(justify left bottom)
-		)
-	)
-	(gr_text "Mousebites for VGA breakout?"
-		(at 148.5138 65.405 90)
-		(layer "User.1")
-		(effects
-			(font
-				(size 1 1)
-				(thickness 0.1)
-			)
-			(justify left bottom)
 		)
 	)
